File: KiCAD/horizontal_counter.kicad_sch (KiCad schematic)
At the start: 14 parts, among them U1 74HC161, U10 74HC04, U11 74HC112, U12 74HC32, U13 74HC173, U14 74HC173, U2 74HC161, U3 74HC161, U4 74HC04, U5 74HC04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

Commit message: updated KiCAD todos
Other:
- note added: "TODO: PE should be disabled"
- note added: "TODO: fix bit numbers"
- note added: "bin(200)='0b11001000'"
- note added: "bin(210)='0b11010010'"
Changed lines of the file:
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@@
+		)
+	)
+	(text "TODO: fix bit numbers"
+		(exclude_from_sim no)
+		(at 72.39 117.602 0)
+		(effects
+			(font
+				(size 1.27 1.27)
+			)
+		)
+	)
+	(text "TODO: PE should be disabled"
+		(exclude_from_sim no)
+		(at 25.4 29.718 0)
+		(effects
+			(font
+				(size 1.27 1.27)
+			)
+		)
+	)
+	(text "bin(210)='0b11010010'"
+		(exclude_from_sim no)
+		(at 120.65 122.682 0)
+		(effects
+			(font
+				(size 1.27 1.27)
+			)
+		)
+	)
+	(text "bin(200)='0b11001000'"
+		(exclude_from_sim no)
+		(at 72.136 91.948 0)
+		(effects
+			(font
+				(size 1.27 1.27)
+			)
 		)
 	)

Commit message: fixed the numbers of horizontal counter NAND gates
Connections:
- net bit_4: now also U8.5
- net bit_5: no longer U8.5
- net bit_6: now also U8.11, U9.11
- net bit_7: now also U8.12, U9.12; no longer U8.11, U9.11
- net bit_8: no longer U8.12, U9.12
- net ~{bit_5}: now also U8.6
- net ~{bit_6}: no longer U8.6
Other:
- note removed: "TODO: fix bit numbers"
Changed lines of the file:
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@@
-		)
-	)
-	(text "TODO: fix bit numbers"
-		(exclude_from_sim no)
-		(at 72.39 117.602 0)
-		(effects
-			(font
-				(size 1.27 1.27)
-			)
 		)
 	)
@@
 	(text "bin(210)='0b11010010'"
 		(exclude_from_sim no)
-		(at 120.65 122.682 0)
+		(at 71.374 118.11 0)
 		(effects
 			(font
@@
 		)
 	)
-	(label "bit_5"
+	(label "bit_4"
 		(at 78.74 132.08 180)
 		(effects
@@
 		)
 	)
-	(label "bit_8"
+	(label "bit_7"
 		(at 78.74 139.7 180)
 		(effects
@@
 		)
 	)
-	(label "bit_7"
+	(label "bit_6"
 		(at 78.74 137.16 180)
 		(effects
@@
 		)
 	)
-	(label "bit_8"
+	(label "bit_7"
 		(at 78.74 115.57 180)
 		(effects
@@
 		)
 	)
-	(label "~{bit_6}"
+	(label "~{bit_5}"
 		(at 78.74 134.62 180)
 		(effects
@@
 		)
 	)
-	(label "bit_7"
+	(label "bit_6"
 		(at 78.74 113.03 180)
 		(effects

Commit message: schematics disabled PE
Connections:
- net +5V: now also U1.9 (~{PE}), U2.9 (~{PE}), U3.9 (~{PE})
- net GND: no longer U1.9 (~{PE}), U2.9 (~{PE}), U3.9 (~{PE})
Other:
- note removed: "TODO: PE should be disabled"
Changed lines of the file:
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@@
-		)
-	)
-	(text "TODO: PE should be disabled"
-		(exclude_from_sim no)
-		(at 25.4 29.718 0)
-		(effects
-			(font
-				(size 1.27 1.27)
-			)
 		)
 	)
@@
 	)
 	(junction
-		(at 120.65 44.45)
-		(diameter 0)
-		(color 0 0 0 0)
-	)
-	(junction
 		(at 259.08 59.69)
 		(diameter 0)
@@
 	)
 	(junction
-		(at 30.48 44.45)
-		(diameter 0)
-		(color 0 0 0 0)
-	)
-	(junction
 		(at 213.36 175.26)
 		(diameter 0)
@@
 	(junction
 		(at 228.6 59.69)
-		(diameter 0)
-		(color 0 0 0 0)
-	)
-	(junction
-		(at 74.93 44.45)
 		(diameter 0)
 		(color 0 0 0 0)
@@
 	(wire
 		(pts
-			(xy 74.93 44.45) (xy 74.93 49.53)
-		)
-		(stroke
-			(width 0)
-			(type default)
-		)
-	)
-	(wire
-		(pts
 			(xy 55.88 49.53) (xy 55.88 57.15)
 		)
@@
 	(wire
 		(pts
+			(xy 30.48 49.53) (xy 30.48 52.07)
+		)
+		(stroke
+			(width 0)
+			(type default)
+		)
+	)
+	(wire
+		(pts
 			(xy 109.22 176.53) (xy 113.03 176.53)
 		)
@@
 	(wire
 		(pts
-			(xy 120.65 44.45) (xy 120.65 49.53)
-		)
-		(stroke
-			(width 0)
-			(type default)
-		)
-	)
-	(wire
-		(pts
 			(xy 168.91 110.49) (xy 168.91 119.38)
 		)
@@
 	(wire
 		(pts
+			(xy 74.93 49.53) (xy 74.93 52.07)
+		)
+		(stroke
+			(width 0)
+			(type default)
+		)
+	)
+	(wire
+		(pts
 			(xy 213.36 113.03) (xy 213.36 114.3)
 		)
@@
 		)
 	)
+	(wire
+		(pts
+			(xy 120.65 49.53) (xy 120.65 52.07)
+		)
+		(stroke
+			(width 0)
+			(type default)
+		)
+	)
 	(bus
 		(pts
@@
 		)
 		(stroke
-			(width 0)
-			(type default)
-		)
-	)
-	(wire
-		(pts
-			(xy 30.48 44.45) (xy 30.48 49.53)
-		)
-		(stroke
